File: KiCadFiles/RC-2XXX/RC-2XXX.kicad_sch (KiCad schematic)
At the start: 155 parts

Commit message: Add new KiCad project files for RC-2XXA, including PCB, schematic, and project files. Update existing schematic for RC-2XXX to adjust paper size and reposition components.
Other:
- moved on the sheet: D1, D10, D11, D12, D13, D14, D15, D16, D17, D18, D19, D2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
