File: KiCadFiles/RC-2XXA/RC-2XXA.kicad_pcb (KiCad board)
At the start: 2 copper layers, 494.6 x 193.6 mm, 282 parts

Commit message: Refactor KiCad project files for RC-2XXA: streamline net connections in PCB, adjust solder mask clearance in project settings, and add new connector symbols in schematic. Enhance error handling for undefined net classes.
Parts:
- removed the D1 at (139.5, 99.2)
- removed the D10 at (311.0, 99.2)
- removed the D11 at (330.0, 99.2)
- removed the D12 at (349.1, 99.2)
- removed the D13 at (139.5, 118.3)
- removed the D14 at (158.6, 118.3)
- removed the D15 at (177.6, 118.3)
- removed the D16 at (196.7, 118.3)
- removed the D17 at (215.7, 118.3)
- removed the D18 at (234.8, 118.3)
- removed the D19 at (253.8, 118.3)
- removed the D2 at (158.6, 99.2)
- removed the D20 at (272.9, 118.3)
- removed the D21 at (291.9, 118.3)
- removed the D22 at (311.0, 118.3)
- removed the D23 at (330.0, 118.3)
- removed the D24 at (349.1, 118.3)
- removed the D3 at (177.6, 99.2)
- removed the D4 at (196.7, 99.2)
- removed the D43 at (411.0, 142.1)
- removed the D44 at (430.0, 142.1)
- removed the D45 at (449.1, 142.1)
- removed the D5 at (215.7, 99.2)
- removed the D6 at (234.8, 99.2)
- removed the D66 at (411.0, 161.1)
- removed the D67 at (430.0, 161.1)
- removed the D68 at (449.1, 161.1)
- removed the D7 at (253.8, 99.2)
- removed the D8 at (272.9, 99.2)
- removed the D9 at (291.9, 99.2)
- removed the D90 at (411.0, 180.2)
- removed the D91 at (430.0, 180.2)
- removed the D92 at (449.1, 180.2)
- removed the MX1 at (136.3, 93.9)
- removed the MX10 at (307.8, 93.9)
- removed the MX11 at (326.8, 93.9)
- removed the MX12 at (345.9, 93.9)
- removed the MX13 at (136.3, 113.0)
- removed the MX14 at (155.4, 113.0)
- removed the MX15 at (174.4, 113.0)
- removed the MX16 at (193.5, 113.0)
- removed the MX17 at (212.5, 113.0)
- removed the MX18 at (231.6, 113.0)
- removed the MX19 at (250.6, 113.0)
- removed the MX2 at (155.4, 93.9)
- removed the MX20 at (269.7, 113.0)
- removed the MX21 at (288.7, 113.0)
- removed the MX22 at (307.8, 113.0)
- removed the MX23 at (326.8, 113.0)
- removed the MX24 at (345.9, 113.0)
- removed the MX3 at (174.4, 93.9)
- removed the MX4 at (193.5, 93.9)
- removed the MX43 at (407.8, 136.8)
- removed the MX44 at (426.9, 136.8)
- removed the MX45 at (445.9, 136.8)
- removed the MX5 at (212.5, 93.9)
- removed the MX6 at (231.6, 93.9)
- removed the MX66 at (407.8, 155.9)
- removed the MX67 at (426.9, 155.9)
- removed the MX68 at (445.9, 155.9)
- removed the MX7 at (250.6, 93.9)
- removed the MX8 at (269.7, 93.9)
- removed the MX9 at (288.7, 93.9)
- removed the MX90 at (407.8, 174.9)
- removed the MX91 at (426.9, 174.9)
- removed the MX92 at (445.9, 174.9)
- D1: renamed from D25; footprint Diode_SMD:D_SOD-323_HandSoldering -> Diode_SMD:D_SOD-123
- D10: renamed from D34; footprint Diode_SMD:D_SOD-323_HandSoldering -> Diode_SMD:D_SOD-123
- D100: renamed from D133; footprint Diode_SMD:D_SOD-323_HandSoldering -> Diode_SMD:D_SOD-123
- D101: renamed from D134; footprint Diode_SMD:D_SOD-323_HandSoldering -> Diode_SMD:D_SOD-123
- D102: renamed from D135; footprint Diode_SMD:D_SOD-323_HandSoldering -> Diode_SMD:D_SOD-123
- D103: renamed from D136; footprint Diode_SMD:D_SOD-323_HandSoldering -> Diode_SMD:D_SOD-123
- D104: renamed from D137; footprint Diode_SMD:D_SOD-323_HandSoldering -> Diode_SMD:D_SOD-123
- D11: renamed from D35; footprint Diode_SMD:D_SOD-323_HandSoldering -> Diode_SMD:D_SOD-123
- D12: renamed from D36; footprint Diode_SMD:D_SOD-323_HandSoldering -> Diode_SMD:D_SOD-123
- D13: renamed from D37; footprint Diode_SMD:D_SOD-323_HandSoldering -> Diode_SMD:D_SOD-123
- D14: renamed from D38; footprint Diode_SMD:D_SOD-323_HandSoldering -> Diode_SMD:D_SOD-123
- D15: renamed from D39; footprint Diode_SMD:D_SOD-323_HandSoldering -> Diode_SMD:D_SOD-123
- D16: renamed from D40; footprint Diode_SMD:D_SOD-323_HandSoldering -> Diode_SMD:D_SOD-123
- D17: renamed from D41; footprint Diode_SMD:D_SOD-323_HandSoldering -> Diode_SMD:D_SOD-123
- D18: renamed from D42; footprint Diode_SMD:D_SOD-323_HandSoldering -> Diode_SMD:D_SOD-123
- D19: renamed from D46; footprint Diode_SMD:D_SOD-323_HandSoldering -> Diode_SMD:D_SOD-123
- D2: renamed from D26; footprint Diode_SMD:D_SOD-323_HandSoldering -> Diode_SMD:D_SOD-123
- D20: renamed from D47; footprint Diode_SMD:D_SOD-323_HandSoldering -> Diode_SMD:D_SOD-123
- D21: renamed from D48; footprint Diode_SMD:D_SOD-323_HandSoldering -> Diode_SMD:D_SOD-123
- D22: renamed from D49; footprint Diode_SMD:D_SOD-323_HandSoldering -> Diode_SMD:D_SOD-123
- D23: renamed from D50; footprint Diode_SMD:D_SOD-323_HandSoldering -> Diode_SMD:D_SOD-123
- D24: renamed from D51; footprint Diode_SMD:D_SOD-323_HandSoldering -> Diode_SMD:D_SOD-123
- D25: renamed from D52; footprint Diode_SMD:D_SOD-323_HandSoldering -> Diode_SMD:D_SOD-123
- D26: renamed from D53; footprint Diode_SMD:D_SOD-323_HandSoldering -> Diode_SMD:D_SOD-123
- D27: renamed from D54; footprint Diode_SMD:D_SOD-323_HandSoldering -> Diode_SMD:D_SOD-123
- D28: renamed from D55; footprint Diode_SMD:D_SOD-323_HandSoldering -> Diode_SMD:D_SOD-123
- D29: renamed from D56; footprint Diode_SMD:D_SOD-323_HandSoldering -> Diode_SMD:D_SOD-123
- D3: renamed from D27; footprint Diode_SMD:D_SOD-323_HandSoldering -> Diode_SMD:D_SOD-123
- D30: renamed from D57; footprint Diode_SMD:D_SOD-323_HandSoldering -> Diode_SMD:D_SOD-123
- D31: renamed from D58; footprint Diode_SMD:D_SOD-323_HandSoldering -> Diode_SMD:D_SOD-123
- D32: renamed from D59; footprint Diode_SMD:D_SOD-323_HandSoldering -> Diode_SMD:D_SOD-123
- D33: renamed from D60; footprint Diode_SMD:D_SOD-323_HandSoldering -> Diode_SMD:D_SOD-123
- D34: renamed from D61; footprint Diode_SMD:D_SOD-323_HandSoldering -> Diode_SMD:D_SOD-123
- D35: renamed from D62; footprint Diode_SMD:D_SOD-323_HandSoldering -> Diode_SMD:D_SOD-123
- D36: renamed from D63; footprint Diode_SMD:D_SOD-323_HandSoldering -> Diode_SMD:D_SOD-123
- D37: renamed from D64; footprint Diode_SMD:D_SOD-323_HandSoldering -> Diode_SMD:D_SOD-123
- D38: renamed from D65; footprint Diode_SMD:D_SOD-323_HandSoldering -> Diode_SMD:D_SOD-123
- D39: renamed from D69; footprint Diode_SMD:D_SOD-323_HandSoldering -> Diode_SMD:D_SOD-123
- D4: renamed from D28; footprint Diode_SMD:D_SOD-323_HandSoldering -> Diode_SMD:D_SOD-123
- D40: renamed from D70; footprint Diode_SMD:D_SOD-323_HandSoldering -> Diode_SMD:D_SOD-123
- D41: renamed from D71; footprint Diode_SMD:D_SOD-323_HandSoldering -> Diode_SMD:D_SOD-123
- D42: renamed from D72; footprint Diode_SMD:D_SOD-323_HandSoldering -> Diode_SMD:D_SOD-123
- D43: renamed from D73; footprint Diode_SMD:D_SOD-323_HandSoldering -> Diode_SMD:D_SOD-123
- D44: renamed from D74; footprint Diode_SMD:D_SOD-323_HandSoldering -> Diode_SMD:D_SOD-123
- D45: renamed from D75; footprint Diode_SMD:D_SOD-323_HandSoldering -> Diode_SMD:D_SOD-123
- D46: renamed from D76; footprint Diode_SMD:D_SOD-323_HandSoldering -> Diode_SMD:D_SOD-123
- D47: renamed from D77; footprint Diode_SMD:D_SOD-323_HandSoldering -> Diode_SMD:D_SOD-123
- D48: renamed from D78; footprint Diode_SMD:D_SOD-323_HandSoldering -> Diode_SMD:D_SOD-123
- D49: renamed from D79; footprint Diode_SMD:D_SOD-323_HandSoldering -> Diode_SMD:D_SOD-123
- D5: renamed from D29; footprint Diode_SMD:D_SOD-323_HandSoldering -> Diode_SMD:D_SOD-123
- D50: renamed from D80; footprint Diode_SMD:D_SOD-323_HandSoldering -> Diode_SMD:D_SOD-123
- D51: renamed from D81; footprint Diode_SMD:D_SOD-323_HandSoldering -> Diode_SMD:D_SOD-123
- D52: renamed from D82; footprint Diode_SMD:D_SOD-323_HandSoldering -> Diode_SMD:D_SOD-123
- D53: renamed from D83; footprint Diode_SMD:D_SOD-323_HandSoldering -> Diode_SMD:D_SOD-123
- D54: renamed from D84; footprint Diode_SMD:D_SOD-323_HandSoldering -> Diode_SMD:D_SOD-123
- D55: renamed from D85; footprint Diode_SMD:D_SOD-323_HandSoldering -> Diode_SMD:D_SOD-123
- D56: renamed from D86; footprint Diode_SMD:D_SOD-323_HandSoldering -> Diode_SMD:D_SOD-123
- D57: renamed from D87; footprint Diode_SMD:D_SOD-323_HandSoldering -> Diode_SMD:D_SOD-123
- D58: renamed from D88; footprint Diode_SMD:D_SOD-323_HandSoldering -> Diode_SMD:D_SOD-123
- D59: renamed from D89; footprint Diode_SMD:D_SOD-323_HandSoldering -> Diode_SMD:D_SOD-123
- D6: renamed from D30; footprint Diode_SMD:D_SOD-323_HandSoldering -> Diode_SMD:D_SOD-123
- D60: renamed from D93; footprint Diode_SMD:D_SOD-323_HandSoldering -> Diode_SMD:D_SOD-123
- D61: renamed from D94; footprint Diode_SMD:D_SOD-323_HandSoldering -> Diode_SMD:D_SOD-123
- D62: renamed from D95; footprint Diode_SMD:D_SOD-323_HandSoldering -> Diode_SMD:D_SOD-123
- D63: renamed from D96; footprint Diode_SMD:D_SOD-323_HandSoldering -> Diode_SMD:D_SOD-123
- D64: renamed from D97; footprint Diode_SMD:D_SOD-323_HandSoldering -> Diode_SMD:D_SOD-123
- D65: renamed from D98; footprint Diode_SMD:D_SOD-323_HandSoldering -> Diode_SMD:D_SOD-123
- D66: renamed from D99; footprint Diode_SMD:D_SOD-323_HandSoldering -> Diode_SMD:D_SOD-123
- D67: renamed from D100; footprint Diode_SMD:D_SOD-323_HandSoldering -> Diode_SMD:D_SOD-123
- D68: renamed from D101; footprint Diode_SMD:D_SOD-323_HandSoldering -> Diode_SMD:D_SOD-123
- D69: renamed from D102; footprint Diode_SMD:D_SOD-323_HandSoldering -> Diode_SMD:D_SOD-123
- D7: renamed from D31; footprint Diode_SMD:D_SOD-323_HandSoldering -> Diode_SMD:D_SOD-123
- D70: renamed from D103; footprint Diode_SMD:D_SOD-323_HandSoldering -> Diode_SMD:D_SOD-123
- D71: renamed from D104; footprint Diode_SMD:D_SOD-323_HandSoldering -> Diode_SMD:D_SOD-123
- D72: renamed from D105; footprint Diode_SMD:D_SOD-323_HandSoldering -> Diode_SMD:D_SOD-123
- D73: renamed from D106; footprint Diode_SMD:D_SOD-323_HandSoldering -> Diode_SMD:D_SOD-123
- D74: renamed from D107; footprint Diode_SMD:D_SOD-323_HandSoldering -> Diode_SMD:D_SOD-123
- D75: renamed from D108; footprint Diode_SMD:D_SOD-323_HandSoldering -> Diode_SMD:D_SOD-123
- D76: renamed from D109; footprint Diode_SMD:D_SOD-323_HandSoldering -> Diode_SMD:D_SOD-123
- D77: renamed from D110; footprint Diode_SMD:D_SOD-323_HandSoldering -> Diode_SMD:D_SOD-123
- D78: renamed from D111; footprint Diode_SMD:D_SOD-323_HandSoldering -> Diode_SMD:D_SOD-123
- D79: renamed from D112; footprint Diode_SMD:D_SOD-323_HandSoldering -> Diode_SMD:D_SOD-123
- D8: renamed from D32; footprint Diode_SMD:D_SOD-323_HandSoldering -> Diode_SMD:D_SOD-123
- D80: renamed from D113; footprint Diode_SMD:D_SOD-323_HandSoldering -> Diode_SMD:D_SOD-123
- D81: renamed from D114; footprint Diode_SMD:D_SOD-323_HandSoldering -> Diode_SMD:D_SOD-123
- D82: renamed from D115; footprint Diode_SMD:D_SOD-323_HandSoldering -> Diode_SMD:D_SOD-123
- D83: renamed from D116; footprint Diode_SMD:D_SOD-323_HandSoldering -> Diode_SMD:D_SOD-123
- D84: renamed from D117; footprint Diode_SMD:D_SOD-323_HandSoldering -> Diode_SMD:D_SOD-123
- D85: renamed from D118; footprint Diode_SMD:D_SOD-323_HandSoldering -> Diode_SMD:D_SOD-123
- D86: renamed from D119; footprint Diode_SMD:D_SOD-323_HandSoldering -> Diode_SMD:D_SOD-123
- D87: renamed from D120; footprint Diode_SMD:D_SOD-323_HandSoldering -> Diode_SMD:D_SOD-123
- D88: renamed from D121; footprint Diode_SMD:D_SOD-323_HandSoldering -> Diode_SMD:D_SOD-123
- D89: renamed from D122; footprint Diode_SMD:D_SOD-323_HandSoldering -> Diode_SMD:D_SOD-123
- D9: renamed from D33; footprint Diode_SMD:D_SOD-323_HandSoldering -> Diode_SMD:D_SOD-123
- D90: renamed from D123; footprint Diode_SMD:D_SOD-323_HandSoldering -> Diode_SMD:D_SOD-123
- D91: renamed from D124; footprint Diode_SMD:D_SOD-323_HandSoldering -> Diode_SMD:D_SOD-123
- D92: renamed from D125; footprint Diode_SMD:D_SOD-323_HandSoldering -> Diode_SMD:D_SOD-123
- D93: renamed from D126; footprint Diode_SMD:D_SOD-323_HandSoldering -> Diode_SMD:D_SOD-123
- D94: renamed from D127; footprint Diode_SMD:D_SOD-323_HandSoldering -> Diode_SMD:D_SOD-123
- D95: renamed from D128; footprint Diode_SMD:D_SOD-323_HandSoldering -> Diode_SMD:D_SOD-123
- D96: renamed from D129; footprint Diode_SMD:D_SOD-323_HandSoldering -> Diode_SMD:D_SOD-123
- D97: renamed from D130; footprint Diode_SMD:D_SOD-323_HandSoldering -> Diode_SMD:D_SOD-123
- D98: renamed from D131; footprint Diode_SMD:D_SOD-323_HandSoldering -> Diode_SMD:D_SOD-123
- D99: renamed from D132; footprint Diode_SMD:D_SOD-323_HandSoldering -> Diode_SMD:D_SOD-123
- moved D28 5.71 mm to (187.3, 164.0)
- moved D32 5.71 mm to (263.5, 164.0)
- moved D33 5.71 mm to (282.6, 164.0)
- moved D34 5.71 mm to (301.6, 164.0)
- moved D37 5.71 mm to (358.8, 164.0)
- moved D38 5.71 mm to (382.6, 164.0)
- moved D40 5.71 mm to (501.6, 164.0)
- moved D101 5.71 mm to (492.1, 221.2)
- moved D102 5.71 mm to (501.6, 221.2)
- moved D13 5.71 mm to (311.1, 145.0)
- moved D14 5.71 mm to (330.2, 145.0)
- moved D15 5.71 mm to (349.2, 145.0)
- moved D17 5.71 mm to (377.8, 145.0)
- moved D20 5.71 mm to (501.6, 145.0)
- moved D4 5.71 mm to (139.7, 145.0)
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- renumbered MX25 to MX1, MX34 to MX10, MX133 to MX100, MX134 to MX101, MX135 to MX102, MX136 to MX103, MX137 to MX104, MX35 to MX11, MX36 to MX12, MX37 to MX13, MX38 to MX14, MX39 to MX15, MX40 to MX16, MX41 to MX17, MX42 to MX18, MX46 to MX19, MX26 to MX2, MX47 to MX20, MX48 to MX21, MX49 to MX22, MX50 to MX23, MX51 to MX24, MX52 to MX25, MX53 to MX26, MX54 to MX27, MX55 to MX28, MX56 to MX29, MX27 to MX3, MX57 to MX30, MX58 to MX31, MX59 to MX32, MX60 to MX33, MX61 to MX34, MX62 to MX35, MX63 to MX36, MX64 to MX37, MX65 to MX38, MX69 to MX39, MX28 to MX4, MX70 to MX40, MX71 to MX41, MX72 to MX42, MX73 to MX43, MX74 to MX44, MX75 to MX45, MX76 to MX46, MX77 to MX47, MX78 to MX48, MX79 to MX49, MX29 to MX5, MX80 to MX50, MX81 to MX51, MX82 to MX52, MX83 to MX53, MX84 to MX54, MX85 to MX55, MX86 to MX56, MX87 to MX57, MX88 to MX58, MX89 to MX59, MX30 to MX6, MX93 to MX60, MX94 to MX61, MX95 to MX62, MX96 to MX63, MX97 to MX64, MX98 to MX65, MX99 to MX66, MX100 to MX67, MX101 to MX68, MX102 to MX69, MX31 to MX7, MX103 to MX70, MX104 to MX71, MX105 to MX72, MX106 to MX73, MX107 to MX74, MX108 to MX75, MX109 to MX76, MX110 to MX77, MX111 to MX78, MX112 to MX79, MX32 to MX8, MX113 to MX80, MX114 to MX81, MX115 to MX82, MX116 to MX83, MX117 to MX84, MX118 to MX85, MX119 to MX86, MX120 to MX87, MX121 to MX88, MX122 to MX89, MX33 to MX9, MX123 to MX90, MX124 to MX91, MX125 to MX92, MX126 to MX93, MX127 to MX94, MX128 to MX95, MX129 to MX96, MX130 to MX97, MX131 to MX98, MX132 to MX99, S134 to S101, S41 to S17, S73 to S43, S89 to S59, S100 to S67, S113 to S80, S122 to S89, S127 to S94

Commit message: Update RC-2XXA KiCad files: adjust footprint properties, correct rectangle positions in schematic, and enhance error handling for pin connections. Remove unnecessary junctions and wires for improved clarity.
Parts:
- moved D41 11.6 mm to (520.8, 152.4)
- moved D23 11.6 mm to (73.2, 152.4)
- moved D24 11.6 mm to (92.2, 152.4)
- moved D25 11.6 mm to (125.5, 152.4)
- moved D26 11.6 mm to (149.4, 152.4)
- moved D27 11.6 mm to (168.4, 152.4)
- moved D28 11.6 mm to (187.5, 152.4)
- moved D29 11.6 mm to (206.5, 152.4)
- moved D30 11.6 mm to (225.6, 152.4)
- moved D31 11.6 mm to (244.6, 152.4)
- moved D32 11.6 mm to (263.7, 152.4)
- moved D33 11.6 mm to (282.7, 152.4)
- moved D34 11.6 mm to (301.8, 152.4)
- moved D35 11.6 mm to (320.8, 152.4)
- moved D36 11.6 mm to (339.9, 152.4)
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
Commit message: updated pcb & sch
Parts:
- added C1: 4.7nF, Capacitor_SMD:C_0805_2012Metric_Pad1.18x1.45mm_HandSolder, F.Cu at (714.2, 160.0)
- added C10: 100nF, Capacitor_SMD:C_0805_2012Metric_Pad1.18x1.45mm_HandSolder, F.Cu at (719.0, 172.0)
- added C11: 10uF, Capacitor_SMD:C_0805_2012Metric_Pad1.18x1.45mm_HandSolder, F.Cu at (723.8, 160.0)
- added C12: 1uF, Capacitor_SMD:C_0805_2012Metric_Pad1.18x1.45mm_HandSolder, F.Cu at (723.8, 163.0)
- added C13: 1uF, Capacitor_SMD:C_0805_2012Metric_Pad1.18x1.45mm_HandSolder, F.Cu at (723.8, 166.0)
- added C2: 1uF, Capacitor_SMD:C_0805_2012Metric_Pad1.18x1.45mm_HandSolder, F.Cu at (714.2, 163.0)
- added C3: 1uF, Capacitor_SMD:C_0805_2012Metric_Pad1.18x1.45mm_HandSolder, F.Cu at (714.2, 166.0)
- added C4: 4.7uF/10V, Capacitor_SMD:C_0805_2012Metric_Pad1.18x1.45mm_HandSolder, F.Cu at (714.2, 169.0)
- added C5: 100nF, Capacitor_SMD:C_0805_2012Metric_Pad1.18x1.45mm_HandSolder, F.Cu at (714.2, 172.0)
- added C6: 100nF, Capacitor_SMD:C_0805_2012Metric_Pad1.18x1.45mm_HandSolder, F.Cu at (719.0, 160.0)
- added C7: 100nF, Capacitor_SMD:C_0805_2012Metric_Pad1.18x1.45mm_HandSolder, F.Cu at (719.0, 163.0)
- added C8: 100nF, Capacitor_SMD:C_0805_2012Metric_Pad1.18x1.45mm_HandSolder, F.Cu at (719.0, 166.0)
- added C9: 100nF, Capacitor_SMD:C_0805_2012Metric_Pad1.18x1.45mm_HandSolder, F.Cu at (719.0, 169.0)
- added F1: 500mA, Fuse:Fuse_1206_3216Metric, F.Cu at (723.1, 215.8)
- added J1: Conn_01x01_Pin, TestPoint:TestPoint_THTPad_2.0x2.0mm_Drill1.0mm, F.Cu at (723.3, 175.5)
- added J2: Conn_01x04_Pin, Connector_JST:JST_SH_SM04B-SRSS-TB_1x04-1MP_P1.00mm_Horizontal, F.Cu at (700.4, 210.7)
- added J3: Conn_01x04_Pin, Connector_PinHeader_1.27mm:PinHeader_1x04_P1.27mm_Vertical, F.Cu at (722.4, 204.2)
- added LED1: LED, My-Fi Footprints:DIP_LED_MX_3mm, F.Cu at (666.0, 207.7)
- added LED2: LED, My-Fi Footprints:DIP_LED_MX_3mm, F.Cu at (671.4, 207.7)
- added LED3: LED, My-Fi Footprints:DIP_LED_MX_3mm, F.Cu at (676.9, 207.7)
- added LED4: LED, My-Fi Footprints:DIP_LED_MX_3mm, F.Cu at (682.3, 207.7)
- added LED5: LED, My-Fi Footprints:DIP_LED_MX_3mm, F.Cu at (687.8, 207.7)
- added LED6: LED, My-Fi Footprints:DIP_LED_MX_3mm, F.Cu at (693.2, 207.7)
- added R1: 1M, Resistor_SMD:R_0805_2012Metric_Pad1.20x1.40mm_HandSolder, F.Cu at (714.1, 175.0)
- added R10: 10k, Resistor_SMD:R_0805_2012Metric_Pad1.20x1.40mm_HandSolder, F.Cu at (718.9, 183.8)
- added R2: 220, Resistor_SMD:R_0805_2012Metric_Pad1.20x1.40mm_HandSolder, F.Cu at (714.1, 177.9)
- added R3: 220, Resistor_SMD:R_0805_2012Metric_Pad1.20x1.40mm_HandSolder, F.Cu at (714.1, 180.9)
- added R4: 10k, Resistor_SMD:R_0805_2012Metric_Pad1.20x1.40mm_HandSolder, F.Cu at (714.1, 183.8)
- added R5: 39R, Resistor_SMD:R_0805_2012Metric_Pad1.20x1.40mm_HandSolder, F.Cu at (714.1, 186.8)
- added R6: 220, Resistor_SMD:R_0805_2012Metric_Pad1.20x1.40mm_HandSolder, F.Cu at (714.1, 189.7)
- added R7: 220, Resistor_SMD:R_0805_2012Metric_Pad1.20x1.40mm_HandSolder, F.Cu at (718.9, 175.0)
- added R8: 220, Resistor_SMD:R_0805_2012Metric_Pad1.20x1.40mm_HandSolder, F.Cu at (718.9, 177.9)
- added R9: 220, Resistor_SMD:R_0805_2012Metric_Pad1.20x1.40mm_HandSolder, F.Cu at (718.9, 180.9)
- added SW1: SW_DPST_x2, Button_Switch_SMD:SW_Push_1P1T_XKB_TS-1187A, F.Cu at (716.0, 205.9)
- added SW2: SW_DPST_x2, Button_Switch_SMD:SW_Push_1P1T_XKB_TS-1187A, F.Cu at (716.0, 212.5)
- added U1: TLV74318PDBVR, Package_TO_SOT_SMD:SOT-23-5, F.Cu at (707.4, 209.3)
- added U2: PMW3360DM-T2QU, My-Fi Footprints:TrackballHolder_34mm, F.Cu at (687.5, 182.7)
- added U3: SRV05-4, Package_TO_SOT_SMD:SOT-23-6, F.Cu at (707.4, 214.0)
- added U4: STM32F072CBTx, Package_QFP:LQFP-48_7x7mm_P0.5mm, F.Cu at (717.4, 196.9)
- added U5: XC6206PxxxMR, Package_TO_SOT_SMD:SOT-23-3, F.Cu at (722.9, 211.9)
Connections:
- D1 pad 1: unconnected-(D1-K-Pad1) -> ROW0
- D10 pad 1: unconnected-(D10-K-Pad1) -> ROW2
- D100 pad 1: unconnected-(D100-K-Pad1) -> ROW6
- D101 pad 1: unconnected-(D101-K-Pad1) -> ROW6
- D102 pad 1: unconnected-(D102-K-Pad1) -> ROW6
- D103 pad 1: unconnected-(D103-K-Pad1) -> ROW6
- D104 pad 1: unconnected-(D104-K-Pad1) -> ROW6
- D11 pad 1: unconnected-(D11-K-Pad1) -> ROW2
- D12 pad 1: unconnected-(D12-K-Pad1) -> ROW2
- D13 pad 1: unconnected-(D13-K-Pad1) -> ROW2
- D14 pad 1: unconnected-(D14-K-Pad1) -> ROW2
- D15 pad 1: unconnected-(D15-K-Pad1) -> ROW2
- D16 pad 1: unconnected-(D16-K-Pad1) -> ROW2
- D17 pad 1: unconnected-(D17-K-Pad1) -> ROW2
- D18 pad 1: unconnected-(D18-K-Pad1) -> ROW2
- D19 pad 1: unconnected-(D19-K-Pad1) -> ROW2
- D2 pad 1: unconnected-(D2-K-Pad1) -> ROW1
- D20 pad 1: unconnected-(D20-K-Pad1) -> ROW2
- D21 pad 1: unconnected-(D21-K-Pad1) -> ROW2
- D22 pad 1: unconnected-(D22-K-Pad1) -> ROW2
- D23 pad 1: unconnected-(D23-K-Pad1) -> ROW0
- D24 pad 1: unconnected-(D24-K-Pad1) -> ROW1
- D25 pad 1: unconnected-(D25-K-Pad1) -> ROW3
- D26 pad 1: unconnected-(D26-K-Pad1) -> ROW3
- D27 pad 1: unconnected-(D27-K-Pad1) -> ROW3
- D28 pad 1: unconnected-(D28-K-Pad1) -> ROW3
- D29 pad 1: unconnected-(D29-K-Pad1) -> ROW3
- D3 pad 1: unconnected-(D3-K-Pad1) -> ROW2
- D30 pad 1: unconnected-(D30-K-Pad1) -> ROW3
- D31 pad 1: unconnected-(D31-K-Pad1) -> ROW3
- D32 pad 1: unconnected-(D32-K-Pad1) -> ROW3
- D33 pad 1: unconnected-(D33-K-Pad1) -> ROW3
- D34 pad 1: unconnected-(D34-K-Pad1) -> ROW3
- D35 pad 1: unconnected-(D35-K-Pad1) -> ROW3
- D36 pad 1: unconnected-(D36-K-Pad1) -> ROW3
- D37 pad 1: unconnected-(D37-K-Pad1) -> ROW3
- D38 pad 1: unconnected-(D38-K-Pad1) -> ROW3
- D39 pad 1: unconnected-(D39-K-Pad1) -> ROW3
- D4 pad 1: unconnected-(D4-K-Pad1) -> ROW2
- D40 pad 1: unconnected-(D40-K-Pad1) -> ROW3
- D41 pad 1: unconnected-(D41-K-Pad1) -> ROW3
- D42 pad 1: unconnected-(D42-K-Pad1) -> ROW3
- D44 pad 1: unconnected-(D44-K-Pad1) -> ROW0
- D45 pad 1: unconnected-(D45-K-Pad1) -> ROW1
- D46 pad 1: unconnected-(D46-K-Pad1) -> ROW4
- D47 pad 1: unconnected-(D47-K-Pad1) -> ROW4
- D48 pad 1: unconnected-(D48-K-Pad1) -> ROW4
- D49 pad 1: unconnected-(D49-K-Pad1) -> ROW4
- D5 pad 1: unconnected-(D5-K-Pad1) -> ROW2
- D50 pad 1: unconnected-(D50-K-Pad1) -> ROW4
- D51 pad 1: unconnected-(D51-K-Pad1) -> ROW4
- D52 pad 1: unconnected-(D52-K-Pad1) -> ROW4
- D53 pad 1: unconnected-(D53-K-Pad1) -> ROW4
- D54 pad 1: unconnected-(D54-K-Pad1) -> ROW4
- D55 pad 1: unconnected-(D55-K-Pad1) -> ROW4
- D56 pad 1: unconnected-(D56-K-Pad1) -> ROW4
- D57 pad 1: unconnected-(D57-K-Pad1) -> ROW4
- D58 pad 1: unconnected-(D58-K-Pad1) -> ROW4
- D59 pad 1: unconnected-(D59-K-Pad1) -> ROW4
- D6 pad 1: unconnected-(D6-K-Pad1) -> ROW2
- D60 pad 1: unconnected-(D60-K-Pad1) -> ROW4
- D61 pad 1: unconnected-(D61-K-Pad1) -> ROW4
- D62 pad 1: unconnected-(D62-K-Pad1) -> ROW4
- D63 pad 1: unconnected-(D63-K-Pad1) -> ROW4
- D64 pad 1: unconnected-(D64-K-Pad1) -> ROW0
- D65 pad 1: unconnected-(D65-K-Pad1) -> ROW1
- D66 pad 1: unconnected-(D66-K-Pad1) -> ROW5
- D67 pad 1: unconnected-(D67-K-Pad1) -> ROW5
- D68 pad 1: unconnected-(D68-K-Pad1) -> ROW5
- D69 pad 1: unconnected-(D69-K-Pad1) -> ROW5
- D7 pad 1: unconnected-(D7-K-Pad1) -> ROW2
- D70 pad 1: unconnected-(D70-K-Pad1) -> ROW5
- D71 pad 1: unconnected-(D71-K-Pad1) -> ROW5
- D72 pad 1: unconnected-(D72-K-Pad1) -> ROW5
- D73 pad 1: unconnected-(D73-K-Pad1) -> ROW5
- D74 pad 1: unconnected-(D74-K-Pad1) -> ROW5
- D75 pad 1: unconnected-(D75-K-Pad1) -> ROW5
- D76 pad 1: unconnected-(D76-K-Pad1) -> ROW5
- D77 pad 1: unconnected-(D77-K-Pad1) -> ROW5
- D78 pad 1: unconnected-(D78-K-Pad1) -> ROW5
- D79 pad 1: unconnected-(D79-K-Pad1) -> ROW5
- D8 pad 1: unconnected-(D8-K-Pad1) -> ROW2
- D80 pad 1: unconnected-(D80-K-Pad1) -> ROW5
- D81 pad 1: unconnected-(D81-K-Pad1) -> ROW5
- D82 pad 1: unconnected-(D82-K-Pad1) -> ROW5
- D83 pad 1: unconnected-(D83-K-Pad1) -> ROW5
- D84 pad 1: unconnected-(D84-K-Pad1) -> ROW5
- D85 pad 1: unconnected-(D85-K-Pad1) -> ROW5
- D86 pad 1: unconnected-(D86-K-Pad1) -> ROW5
- D87 pad 1: unconnected-(D87-K-Pad1) -> ROW5
- D88 pad 1: unconnected-(D88-K-Pad1) -> ROW5
- D9 pad 1: unconnected-(D9-K-Pad1) -> ROW2
- D90 pad 1: unconnected-(D90-K-Pad1) -> ROW0
- D91 pad 1: unconnected-(D91-K-Pad1) -> ROW1
- D92 pad 1: unconnected-(D92-K-Pad1) -> ROW6
- D93 pad 1: unconnected-(D93-K-Pad1) -> ROW6
- D94 pad 1: unconnected-(D94-K-Pad1) -> ROW6
- D95 pad 1: unconnected-(D95-K-Pad1) -> ROW6
- D96 pad 1: unconnected-(D96-K-Pad1) -> ROW6
- D97 pad 1: unconnected-(D97-K-Pad1) -> ROW6
- D98 pad 1: unconnected-(D98-K-Pad1) -> ROW6
- D99 pad 1: unconnected-(D99-K-Pad1) -> ROW6
- MX1 pad 1: unconnected-(MX1-Pad1) -> COL12
- MX10 pad 1: unconnected-(MX10-Pad1) -> COL7
- MX100 pad 1: unconnected-(MX100-Pad1) -> COL17
- MX102 pad 1: unconnected-(MX102-Pad1) -> COL18
- MX103 pad 1: unconnected-(MX103-Pad1) -> COL19
- MX104 pad 1: unconnected-(MX104-Pad1) -> COL20
- MX11 pad 1: unconnected-(MX11-Pad1) -> COL8
- MX12 pad 1: unconnected-(MX12-Pad1) -> COL9
- MX13 pad 1: unconnected-(MX13-Pad1) -> COL10
- MX14 pad 1: unconnected-(MX14-Pad1) -> COL11
- MX15 pad 1: unconnected-(MX15-Pad1) -> COL12
- MX16 pad 1: unconnected-(MX16-Pad1) -> COL13
- MX18 pad 1: unconnected-(MX18-Pad1) -> COL14
- MX19 pad 1: unconnected-(MX19-Pad1) -> COL17
- MX2 pad 1: unconnected-(MX2-Pad1) -> COL12
- MX20 pad 1: unconnected-(MX20-Pad1) -> COL18
- MX21 pad 1: unconnected-(MX21-Pad1) -> COL19
- MX22 pad 1: unconnected-(MX22-Pad1) -> COL20
- MX23 pad 1: unconnected-(MX23-Pad1) -> COL13
- MX24 pad 1: unconnected-(MX24-Pad1) -> COL13
- MX25 pad 1: unconnected-(MX25-Pad1) -> COL0
- MX26 pad 1: unconnected-(MX26-Pad1) -> COL1
- MX27 pad 1: unconnected-(MX27-Pad1) -> COL2
- MX28 pad 1: unconnected-(MX28-Pad1) -> COL3
- MX29 pad 1: unconnected-(MX29-Pad1) -> COL4
- MX3 pad 1: unconnected-(MX3-Pad1) -> COL0
- MX30 pad 1: unconnected-(MX30-Pad1) -> COL5
- MX31 pad 1: unconnected-(MX31-Pad1) -> COL6
- MX32 pad 1: unconnected-(MX32-Pad1) -> COL7
- MX33 pad 1: unconnected-(MX33-Pad1) -> COL8
- MX34 pad 1: unconnected-(MX34-Pad1) -> COL9
- MX35 pad 1: unconnected-(MX35-Pad1) -> COL10
- MX36 pad 1: unconnected-(MX36-Pad1) -> COL11
- MX37 pad 1: unconnected-(MX37-Pad1) -> COL12
- MX38 pad 1: unconnected-(MX38-Pad1) -> COL13
- MX39 pad 1: unconnected-(MX39-Pad1) -> COL17
- MX4 pad 1: unconnected-(MX4-Pad1) -> COL1
- MX40 pad 1: unconnected-(MX40-Pad1) -> COL18
- MX41 pad 1: unconnected-(MX41-Pad1) -> COL19
- MX42 pad 1: unconnected-(MX42-Pad1) -> COL20
- MX43 pad 1: unconnected-(MX43-Pad1) -> COL20
- MX44 pad 1: unconnected-(MX44-Pad1) -> COL14
- MX45 pad 1: unconnected-(MX45-Pad1) -> COL14
- MX46 pad 1: unconnected-(MX46-Pad1) -> COL0
- MX48 pad 1: unconnected-(MX48-Pad1) -> COL1
- MX49 pad 1: unconnected-(MX49-Pad1) -> COL2
- MX5 pad 1: unconnected-(MX5-Pad1) -> COL2
- MX50 pad 1: unconnected-(MX50-Pad1) -> COL3
- MX51 pad 1: unconnected-(MX51-Pad1) -> COL4
- MX52 pad 1: unconnected-(MX52-Pad1) -> COL5
- MX53 pad 1: unconnected-(MX53-Pad1) -> COL6
- MX54 pad 1: unconnected-(MX54-Pad1) -> COL7
- MX55 pad 1: unconnected-(MX55-Pad1) -> COL8
- MX56 pad 1: unconnected-(MX56-Pad1) -> COL9
- MX57 pad 1: unconnected-(MX57-Pad1) -> COL10
- MX58 pad 1: unconnected-(MX58-Pad1) -> COL11
- MX59 pad 1: unconnected-(MX59-Pad1) -> COL12
- MX6 pad 1: unconnected-(MX6-Pad1) -> COL3
- MX60 pad 1: unconnected-(MX60-Pad1) -> COL17
- MX61 pad 1: unconnected-(MX61-Pad1) -> COL18
- MX62 pad 1: unconnected-(MX62-Pad1) -> COL19
- MX63 pad 1: unconnected-(MX63-Pad1) -> COL20
- MX64 pad 1: unconnected-(MX64-Pad1) -> COL15
- MX65 pad 1: unconnected-(MX65-Pad1) -> COL15
- MX66 pad 1: unconnected-(MX66-Pad1) -> COL0
- MX68 pad 1: unconnected-(MX68-Pad1) -> COL1
- MX69 pad 1: unconnected-(MX69-Pad1) -> COL2
- MX7 pad 1: unconnected-(MX7-Pad1) -> COL4
- MX70 pad 1: unconnected-(MX70-Pad1) -> COL3
- MX71 pad 1: unconnected-(MX71-Pad1) -> COL4
- MX72 pad 1: unconnected-(MX72-Pad1) -> COL5
- MX73 pad 1: unconnected-(MX73-Pad1) -> COL6
- MX74 pad 1: unconnected-(MX74-Pad1) -> COL7
- MX75 pad 1: unconnected-(MX75-Pad1) -> COL8
- MX76 pad 1: unconnected-(MX76-Pad1) -> COL9
- MX77 pad 1: unconnected-(MX77-Pad1) -> COL10
- MX78 pad 1: unconnected-(MX78-Pad1) -> COL11
- MX79 pad 1: unconnected-(MX79-Pad1) -> COL12
- MX8 pad 1: unconnected-(MX8-Pad1) -> COL5
- MX81 pad 1: unconnected-(MX81-Pad1) -> COL13
- MX82 pad 1: unconnected-(MX82-Pad1) -> COL14
- MX83 pad 1: unconnected-(MX83-Pad1) -> COL15
- MX84 pad 1: unconnected-(MX84-Pad1) -> COL16
- MX85 pad 1: unconnected-(MX85-Pad1) -> COL17
- MX86 pad 1: unconnected-(MX86-Pad1) -> COL18
- MX87 pad 1: unconnected-(MX87-Pad1) -> COL19
- MX88 pad 1: unconnected-(MX88-Pad1) -> COL20
- MX89 pad 1: unconnected-(MX89-Pad1) -> COL20
- MX9 pad 1: unconnected-(MX9-Pad1) -> COL6
- MX90 pad 1: unconnected-(MX90-Pad1) -> COL16
- MX91 pad 1: unconnected-(MX91-Pad1) -> COL16
- MX92 pad 1: unconnected-(MX92-Pad1) -> COL0
- MX93 pad 1: unconnected-(MX93-Pad1) -> COL3
- MX94 pad 1: unconnected-(MX94-Pad1) -> COL6
- MX95 pad 1: unconnected-(MX95-Pad1) -> COL11
- MX96 pad 1: unconnected-(MX96-Pad1) -> COL13
- MX97 pad 1: unconnected-(MX97-Pad1) -> COL14
- MX98 pad 1: unconnected-(MX98-Pad1) -> COL15
- MX99 pad 1: unconnected-(MX99-Pad1) -> COL16

Commit message: feat(kicad): sync RC-2XXA schematic/PCB and add routing presets
Parts:
- removed D101, D17, D43, D47, D67, D79, D89: 1N4148, Diode_SMD:D_SOD-123
- added D206: SMF6.0A, My-Fi Footprints:D_SOD-123, F.Cu at (714.2, 220.1)
- D1, D10, D100, D102, D103, D104, D11, D12, D13, D14, D15, D16, D18, D19, D2, D20, D21, D22, D23, D24, D25, D26, D27, D28, D29, D3, D30, D31, D32, D33, D34, D35, D36, D37, D38, D39, D4, D40, D41, D42, D44, D45, D46, D48, D49, D5, D50, D51, D52, D53, D54, D55, D56, D57, D58, D59, D6, D60, D61, D62, D63, D64, D65, D66, D68, D69, D7, D70, D71, D72, D73, D74, D75, D76, D77, D78, D8, D80, D81, D82, D83, D84, D85, D86, D87, D88, D9, D90, D91, D92, D93, D94, D95, D96, D97, D98, D99: footprint Diode_SMD:D_SOD-123 -> My-Fi Footprints:D_SOD-123-g
- U3: value SRV05-4 -> TPD4E05U06DQAR; footprint Package_TO_SOT_SMD:SOT-23-6 -> My-Fi Footprints:USON-10_2.5x1.0mm_P0.5mm
- moved U2 262.1 mm to (426.9, 155.9)
- moved J3 35.0 mm to (688.3, 196.3)
- moved J1 34.9 mm to (689.4, 183.5)
- moved LED1 23.2 mm to (642.9, 205.9)
- moved LED2 23.2 mm to (648.3, 205.9)
- moved LED3 23.2 mm to (653.8, 205.9)
- moved LED4 23.2 mm to (659.2, 205.9)
- moved LED5 23.2 mm to (664.6, 205.9)
- moved LED6 23.2 mm to (670.1, 205.9)
- moved D100 18.0 mm to (464.7, 209.6)
- moved U3 11.3 mm to (712.5, 224.1)
- moved D16 8.77 mm to (372.4, 141.2)
- moved D42 7.00 mm to (539.9, 159.4)
- moved D66 7.00 mm to (120.8, 197.5)
- moved D88 7.00 mm to (539.9, 197.5)
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Connections:
- MX101 pad 1: unconnected-(MX101-Pad1) -> COL17
- MX101 pad 2: Net-(D101-A) -> Net-(D100-A)
- MX17 pad 1: unconnected-(MX17-Pad1) -> COL13
- MX17 pad 2: Net-(D17-A) -> Net-(D16-A)
- MX43 pad 2: Net-(D43-A) -> Net-(D42-A)
- MX47 pad 1: unconnected-(MX47-Pad1) -> COL0
- MX47 pad 2: Net-(D47-A) -> Net-(D46-A)
- MX67 pad 1: unconnected-(MX67-Pad1) -> COL1
- MX67 pad 2: Net-(D67-A) -> Net-(D68-A)
- MX79 pad 2: Net-(D79-A) -> Net-(D80-A)
- MX80 pad 1: unconnected-(MX80-Pad1) -> COL12
- MX89 pad 2: Net-(D89-A) -> Net-(D88-A)
- U3 pad 1: unconnected-(U3-IO1-Pad1) -> DP
- U3 pad 2: GND -> DN
- U3 pad 3: unconnected-(U3-IO2-Pad3) -> GND
- U3 pad 4: DN -> DP
- U3 pad 5: +5V -> DN
- U3 pad 6: DP -> DN
Routing:
- net ROW1: track 0.00 -> 83.6 mm
- net ROW0: track 0.00 -> 82.7 mm
- net ROW5: track 0.00 -> 52.2 mm
- net ROW4: track 0.00 -> 37.1 mm
- net ROW2: track 0.00 -> 27.9 mm
- net ROW3: track 0.00 -> 25.2 mm
- net Net-(D100-A): track 0.00 -> 22.3 mm
- net COL16: track 0.00 -> 19.0 mm
- net COL15: track 0.00 -> 19.0 mm
- net COL14: track 0.00 -> 19.0 mm
- net COL13: track 0.00 -> 19.0 mm
- net COL12: track 0.00 -> 19.0 mm
- net Net-(D16-A): track 0.00 -> 17.4 mm
- net Net-(D42-A): track 0.00 -> 16.8 mm
- net Net-(D88-A): track 0.00 -> 16.7 mm
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
Commit message: Refactor code structure for improved readability and maintainability
Parts:
- added J4: Conn_01x07_Socket, Connector_JST:JST_SH_SM07B-SRSS-TB_1x07-1MP_P1.00mm_Horizontal, B.Cu at (215.2, 49.6)
- added J5: Conn_01x07_Socket, Connector_JST:JST_SH_SM07B-SRSS-TB_1x07-1MP_P1.00mm_Horizontal, B.Cu at (271.2, 50.3)
- C1, C10, C11, C12, C13, C2, C3, C4, C5, C6, C7, C8, C9, D206, F1, J2, R1, R10, R2, R3, R4, R5, R6, R7, R8, R9, SW1, SW2, U1, U3, U4, U5: moved to B.Cu
- LED3: footprint My-Fi Footprints:DIP_LED_MX_3mm -> My-Fi Footprints:CAPS_LED_MX_3mm
- moved U3 620.2 mm to (117.2, 49.9), turned to 180 degrees
- moved J3 612.4 mm to (93.1, 52.3)
- moved J1 598.1 mm to (109.1, 38.6)
- moved J2 579.4 mm to (128.1, 85.8), turned to 90 degrees
- moved LED3 535.0 mm to (119.7, 174.9)
- moved LED1 534.8 mm to (112.5, 136.8)
- moved LED6 231.9 mm to (477.5, 76.7)
- moved D206 222.0 mm to (632.6, 13.7), turned to 180 degrees
- moved LED4 203.1 mm to (502.5, 76.7)
- moved LED5 202.3 mm to (474.5, 136.8)
- moved LED2 176.9 mm to (527.5, 76.7)
- moved U4 145.1 mm to (627.2, 83.3), turned to 180 degrees
- moved U5 124.6 mm to (639.7, 119.1), turned to 180 degrees
- moved C11 111.7 mm to (651.3, 75.0), turned to 180 degrees
- moved C12 111.7 mm to (651.3, 78.0), turned to 180 degrees
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Routing:
- net ROW4: track 37.1 -> 620.4 mm
- net ROW3: track 25.2 -> 596.7 mm
- net ROW2: track 27.9 -> 572.6 mm
- net ROW5: track 52.2 -> 581.6 mm
- net ROW6: track 10.6 -> 502.9 mm
- net COL13: track 19.0 -> 122.5 mm
- net COL14: track 19.0 -> 113.2 mm
- net COL6: track 0.00 -> 92.5 mm
- net COL3: track 0.00 -> 91.0 mm
- net COL1: track 0.00 -> 90.5 mm
- net COL17: track 0.00 -> 89.7 mm
- net COL11: track 0.00 -> 87.1 mm
- net COL0: track 0.00 -> 86.9 mm
- net COL12: track 19.0 -> 104.1 mm
- net COL20: track 0.00 -> 79.5 mm
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Other:
- outline, holes or cut-outs redrawn

Commit message: Implement code changes to enhance functionality and improve performance
Parts:
- moved R2 556.1 mm to (107.0, 141.9)
- moved R1 549.0 mm to (112.8, 59.2)
- moved F1 545.9 mm to (111.9, 51.2)
- moved C1 543.0 mm to (118.2, 59.2)
- moved R6 541.8 mm to (124.4, 180.0), turned to 0 degrees
- moved D206 510.8 mm to (122.8, 44.9)
- moved C12 291.5 mm to (360.7, 56.1), turned to -90 degrees
- moved C13 282.0 mm to (370.4, 57.1), turned to -90 degrees
- moved U5 281.4 mm to (365.7, 55.1)
- moved C9 272.2 mm to (384.6, 65.9)
- moved C8 263.9 mm to (392.3, 78.9), turned to -90 degrees
- moved C10 260.1 mm to (397.7, 57.5), turned to 90 degrees
- moved C4 256.6 mm to (415.6, 159.0), turned to -90 degrees
- moved C5 253.4 mm to (418.0, 159.0), turned to -90 degrees
- moved C7 249.7 mm to (406.6, 69.3), turned to 0 degrees
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Routing:
- net +3V3: track 0.00 -> 48.9 mm
- net VDD_TR: track 0.00 -> 25.8 mm
- net Net-(LED3-A): track 0.00 -> 9.37 mm
- net Net-(U2-VDDPIX): track 0.00 -> 5.90 mm
- net +5V: track 0.00 -> 3.88 mm
- net ROW2: track 572.6 -> 576.2 mm
- net Net-(U2-LED_P): track 0.00 -> 3.48 mm
- net MISO: track 0.00 -> 3.39 mm
- net Net-(LED1-A): track 0.00 -> 3.21 mm
- net RST-1: track 0.00 -> 3.15 mm
- net BOOT-1: track 0.00 -> 3.12 mm
- net Net-(LED5-A): track 0.00 -> 3.04 mm

Commit message: Update RC-2XXA project files: Adjust minimum clearance and modify connector properties
- Changed minimum clearance in RC-2XXA.kicad_pro from 0.5 to 0.26.
- Updated the "Value" property of a component in RC-2XXA.kicad_sch from "VBUS" to "+5V".
- Added a new connector symbol with detailed properties including reference, value, footprint, and description.
- Removed the old connector symbol to avoid duplication.
Parts:
- J3: footprint Connector_PinHeader_1.27mm:PinHeader_1x04_P1.27mm_Vertical -> My-Fi Footprints:My-SolderWire-0.5sqmm_1x04_D0.9mm_OD2.1mm; moved to B.Cu
- moved J4 49.6 mm to (165.7, 51.7)
- moved J5 46.9 mm to (318.1, 51.7)
- moved J3 43.4 mm to (125.9, 80.7), turned to 90 degrees
- moved D206 40.9 mm to (139.4, 82.3), turned to -90 degrees
- moved J2 39.4 mm to (165.7, 97.5)
- moved F1 37.3 mm to (134.7, 80.7), turned to 0 degrees
- moved U3 30.9 mm to (134.7, 75.4)
- moved R1 13.2 mm to (118.0, 47.1), turned to 0 degrees
- moved J1 10.8 mm to (114.2, 48.2)
- moved C1 9.73 mm to (118.0, 49.5), turned to 0 degrees
Connections:
- J2 pad 1: VBUS -> +5V
Routing:
- net DN: track 0.00 -> 501.3 mm
- net DP: track 0.00 -> 489.7 mm
- net +5V: track 3.88 -> 466.1 mm, vias 0 -> 6
- net +3V3: track 48.9 -> 74.2 mm
- net GND: track 0.00 -> 9.23 mm
- net GNDREF: track 0.00 -> 9.07 mm
- net VBUS: track 0.00 -> 7.45 mm
- net RST-1: track 3.15 -> 9.15 mm
- net BOOT-1: track 3.12 -> 9.12 mm
- net Net-(LED6-A): track 0.00 -> 5.34 mm
- net Net-(LED2-A): track 0.00 -> 5.08 mm
- net Net-(LED4-A): track 0.00 -> 5.05 mm
Other:
- outline, holes or cut-outs redrawn
- board text added: "Boot"
- board text added: "Reset"
