File: KiCadFiles/RC-2XXA/RC-2XXA.kicad_pcb (KiCad board)
At the start: 2 copper layers, 494.6 x 193.6 mm, 252 parts, among them J1 Conn_01x01_Pin, J2 Conn_01x04_Pin, J3 Conn_01x04_Pin, J4 Conn_01x07_Socket, J5 Conn_01x07_Socket, SW1 SW_DPST_x2, SW2 SW_DPST_x2, U1 TLV74318PDBVR, U2 PMW3360DM-T2QU, U3 TPD4E05U06DQAR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

Commit message: Add Solder Jumper component and associated wiring to RC-2XXA schematic
- Introduced a new Solder Jumper component (JP) with properties including reference, value, footprint, and description.
- Added multiple instances of the Solder Jumper at specified coordinates in the schematic.
- Updated wiring to accommodate the new component, ensuring proper connections.
Parts:
- added JP1: SolderJumper_2_Open, Jumper:SolderJumper-2_P1.3mm_Open_RoundedPad1.0x1.5mm, B.Cu at (519.2, 88.9)
- added JP2: SolderJumper_2_Open, Jumper:SolderJumper-2_P1.3mm_Open_RoundedPad1.0x1.5mm, B.Cu at (494.2, 88.9)
- added JP3: SolderJumper_2_Open, Jumper:SolderJumper-2_P1.3mm_Open_RoundedPad1.0x1.5mm, B.Cu at (468.9, 88.9)
- moved C2 9.09 mm to (433.7, 72.7), turned to 0 degrees
- moved C9 6.58 mm to (383.4, 59.4), turned to 90 degrees
- moved SW1 0.28 mm to (439.5, 58.0)
- moved C6 0.18 mm to (445.6, 57.1)
- moved SW2 0.05 mm to (454.3, 58.0)
Connections:
- R3 pad 2: SCLLED -> Net-(JP1-B)
- R7 pad 2: CAPLED -> Net-(JP2-B)
- R9 pad 2: NUMLED -> Net-(JP3-B)
Routing:
- net SCLLED: track 0.00 -> 584.7 mm, vias 0 -> 8
- net CAPLED: track 0.00 -> 537.2 mm, vias 0 -> 6
- net +3V3: track 74.2 -> 333.5 mm, vias 0 -> 5
- net NUMLED: track 0.00 -> 160.6 mm, vias 0 -> 2
- net VDD_TR: track 25.8 -> 138.2 mm, vias 0 -> 2
- net CS: track 0.00 -> 109.5 mm, vias 0 -> 1
- net MISO: track 3.39 -> 109.5 mm, vias 0 -> 2
- net MOSI: track 0.00 -> 103.1 mm, vias 0 -> 2
- net SCLK: track 0.00 -> 102.3 mm, vias 0 -> 2
- net BOOT-1: track 9.12 -> 75.1 mm, vias 0 -> 2
- net RST-1: track 9.15 -> 51.2 mm, vias 0 -> 2
- net Net-(JP1-B): track 0.00 -> 6.53 mm
- net Net-(JP2-B): track 0.00 -> 6.52 mm
- net Net-(JP3-B): track 0.00 -> 6.50 mm
- net unconnected-(U4-PA13-Pad34): track 0.00 -> 3.32 mm
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
Commit message: Add Mounting Hole Pad and GND symbol to schematic
- Introduced a new symbol for a mounting hole pad with properties including reference, value, footprint, and description.
- Added a graphical representation of the mounting hole pad with a circle.
- Included a GND symbol with properties for reference, value, and description, creating a global label for ground.
- Updated the schematic layout to accommodate the new components.
Parts:
- added H1: MountingHole_Pad, My-Fi Footprints:Cherry-GND-PAD, F.Cu at (138.4, 48.2)
- moved C1 9.85 mm to (112.8, 41.1)
- moved J1 9.85 mm to (109.0, 39.8)
- moved R1 9.85 mm to (112.8, 38.7)
Routing:
- net COL16: track 39.1 -> 611.6 mm, vias 0 -> 3
- net COL15: track 38.7 -> 571.0 mm, vias 0 -> 3
- net COL14: track 113.2 -> 496.0 mm, vias 0 -> 2
- net ROW0: track 82.7 -> 450.2 mm, vias 0 -> 2
- net ROW1: track 83.6 -> 432.0 mm, vias 0 -> 2
- net COL0: track 86.9 -> 429.9 mm, vias 0 -> 1
- net COL13: track 122.5 -> 460.6 mm, vias 0 -> 2
- net COL5: track 67.5 -> 390.2 mm, vias 0 -> 1
- net COL1: track 90.5 -> 412.2 mm, vias 0 -> 1
- net COL2: track 67.6 -> 370.0 mm, vias 0 -> 1
- net COL12: track 104.1 -> 400.0 mm, vias 0 -> 2
- net COL6: track 92.5 -> 386.8 mm, vias 0 -> 1
- net COL3: track 91.0 -> 375.6 mm, vias 0 -> 1
- net COL4: track 67.5 -> 342.5 mm, vias 0 -> 1
- net COL7: track 67.6 -> 317.4 mm, vias 0 -> 1
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Other:
- outline, holes or cut-outs redrawn

Commit message: Add Solder Jumper and update component positions in schematic
- Introduced a new Solder Jumper component (JP4) with properties and graphical representation.
- Adjusted positions of several components including resistors (R8, R9, R11) and LEDs (LED6, LED7) for better layout.
- Updated junctions and wire connections to reflect new component placements.
- Removed redundant junctions and wires to clean up the schematic.
Parts:
- added JP4: SolderJumper_3_Open, Jumper:SolderJumper-3_P1.3mm_Open_RoundedPad1.0x1.5mm, B.Cu at (484.1, 128.4)
- added LED7: LED, My-Fi Footprints:DIP_LED_MX_3mm, F.Cu at (493.5, 136.8)
- added R11: 220, Resistor_SMD:R_0805_2012Metric_Pad1.20x1.40mm_HandSolder, B.Cu at (488.2, 141.9)
- moved C10 7.50 mm to (404.5, 60.6), turned to 0 degrees
- moved C11 3.56 mm to (404.5, 62.8)
- moved C8 3.44 mm to (390.2, 76.1)
- moved C7 1.48 mm to (407.5, 70.5)
Connections:
- JP3 pad 1: NUMLED -> Net-(JP3-A)
- R8 pad 2: NUMLED -> Net-(JP3-A)
Routing:
- net ROW6: track 502.9 -> 615.5 mm, vias 0 -> 3
- net ROW5: track 581.6 -> 675.4 mm, vias 0 -> 1
- net COL20: track 79.5 -> 159.0 mm
- net COL15: track 571.0 -> 636.0 mm
- net COL16: track 611.6 -> 675.7 mm
- net COL12: track 400.0 -> 462.6 mm
- net COL19: track 78.1 -> 138.3 mm
- net COL13: track 460.6 -> 509.4 mm
- net COL14: track 496.0 -> 540.7 mm
- net COL18: track 78.3 -> 121.8 mm
- net COL17: track 89.7 -> 129.1 mm
- net Net-(JP3-A): track 0.00 -> 26.8 mm
- net GND: track 11.6 -> 34.2 mm, vias 1 -> 10
- net Net-(JP4-B): track 0.00 -> 14.3 mm
- net NUMLED: track 160.6 -> 172.9 mm
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